Commit message: updated URDF and ROSClient

File: mecademic_description/urdf/meca_500_r3.urdf.xacro (robot description, xacro)
@@ -1,3 +1,10 @@
 <robot name="meca_500_r3" xmlns:xacro="http://ros.org/wiki/xacro">
+  <!-- FLANGE -->
+  <link name="meca_brf" />
+  <joint name="meca_base_joint" type="fixed">
+    <parent link="meca_brf" />
+    <child link="meca_base_link" />
+    <origin xyz="-0.012 0 0" rpy="0 0 0" />
+  </joint>
   <!-- Base link is the center of the robot's bottom plate -->
   <link name="meca_base_link">
@@ -147,3 +154,10 @@
     <limit effort="10.0" velocity="8.72665" lower="-3.14159" upper="3.14159" />
   </joint>
+  <!-- FLANGE -->
+  <link name="meca_flange_link" />
+  <joint name="meca_flange_joint" type="fixed">
+    <parent link="meca_axis_6_link" />
+    <child link="meca_flange_link" />
+    <origin xyz="0 0 0" rpy="0 ${pi/2} 0" />
+  </joint>
 </robot>

Commit message: Using ROS-like interface

File: mecademic_description/urdf/meca_500_r3.urdf.xacro (robot description, xacro)
@@ -1,163 +1,9 @@
-<robot name="meca_500_r3" xmlns:xacro="http://ros.org/wiki/xacro">
-  <!-- FLANGE -->
-  <link name="meca_brf" />
-  <joint name="meca_base_joint" type="fixed">
-    <parent link="meca_brf" />
-    <child link="meca_base_link" />
-    <origin xyz="-0.012 0 0" rpy="0 0 0" />
-  </joint>
-  <!-- Base link is the center of the robot's bottom plate -->
-  <link name="meca_base_link">
-    <visual>
-      <origin xyz="0 0 0" rpy="0 0 0" />
-      <geometry>
-        <mesh filename="package://mecademic_description/meshes/meca_500_r3_base.dae" />
-      </geometry>
-    </visual>
-    <collision>
-      <origin xyz="0 0 0" rpy="0 0 0" />
-      <geometry>
-        <mesh filename="package://mecademic_description/meshes/meca_500_r3_base_collision.stl" />
-      </geometry>
-    </collision>
-  </link>
-  <!-- Joint 1 -->
-  <link name="meca_axis_1_link">
-    <visual>
-      <origin xyz="0 0 0" rpy="0 0 0" />
-      <geometry>
-        <mesh filename="package://mecademic_description/meshes/meca_500_r3_j1.dae" />
-      </geometry>
-    </visual>
-    <collision>
-      <origin xyz="0 0 0" rpy="0 0 0" />
-      <geometry>
-        <mesh filename="package://mecademic_description/meshes/meca_500_r3_j1_collision.stl" />
-      </geometry>
-    </collision>
-  </link>
-  <joint name="meca_axis_1_joint" type="revolute">
-    <origin xyz="0.012498 0 0.091" rpy="0 0 0" />
-    <parent link="meca_base_link" />
-    <child link="meca_axis_1_link" />
-    <axis xyz="0 0 1" />
-    <limit effort="10.0" velocity="2.61799" lower="-3.05433" upper="3.05433" />
-  </joint>
-  <!-- Joint 2 -->
-  <link name="meca_axis_2_link">
-    <visual>
-      <origin xyz="0 0 0" rpy="0 0 0" />
-      <geometry>
-        <mesh filename="package://mecademic_description/meshes/meca_500_r3_j2.dae" />
-      </geometry>
-    </visual>
-    <collision>
-      <origin xyz="0 0 0" rpy="0 0 0" />
-      <geometry>
-        <mesh filename="package://mecademic_description/meshes/meca_500_r3_j2_collision.stl" />
-      </geometry>
-    </collision>
-  </link>
-  <joint name="meca_axis_2_joint" type="revolute">
-    <origin xyz="0 0 0.044" rpy="0 0 0" />
-    <parent link="meca_axis_1_link" />
-    <child link="meca_axis_2_link" />
-    <axis xyz="0 1 0" />
-    <limit effort="10.0" velocity="2.61799" lower="-1.22173048" upper="1.5708" />
-  </joint>
-  <!-- Joint 3 -->
-  <link name="meca_axis_3_link">
-    <visual>
-      <origin xyz="0 0 0" rpy="0 0 0" />
-      <geometry>
-        <mesh filename="package://mecademic_description/meshes/meca_500_r3_j3.dae" />
-      </geometry>
-    </visual>
-    <collision>
-      <origin xyz="0 0 0" rpy="0 0 0" />
-      <geometry>
-        <mesh filename="package://mecademic_description/meshes/meca_500_r3_j3_collision.stl" />
-      </geometry>
-    </collision>
-  </link>
-  <joint name="meca_axis_3_joint" type="revolute">
-    <origin xyz="0 0 0.135" rpy="0 0 0" />
-    <parent link="meca_axis_2_link" />
-    <child link="meca_axis_3_link" />
-    <axis xyz="0 1 0" />
-    <limit effort="10.0" velocity="3.14159" lower="-2.35619" upper="1.22173048" />
-  </joint>
-  <!-- Joint 4 -->
-  <link name="meca_axis_4_link">
-    <visual>
-      <origin xyz="0 0 0" rpy="0 0 0" />
-      <geometry>
-        <mesh filename="package://mecademic_description/meshes/meca_500_r3_j4.dae" />
-      </geometry>
-    </visual>
-    <collision>
-      <origin xyz="0 0 0" rpy="0 0 0" />
-      <geometry>
-        <mesh filename="package://mecademic_description/meshes/meca_500_r3_j4_collision.stl" />
-      </geometry>
-    </collision>
-  </link>
-  <joint name="meca_axis_4_joint" type="revolute">
-    <origin xyz="0 0 0.038" rpy="0 0 0" />
-    <parent link="meca_axis_3_link" />
-    <child link="meca_axis_4_link" />
-    <axis xyz="1 0 0" />
-    <limit effort="10.0" velocity="5.23599" lower="-2.96706" upper="2.96706" />
-  </joint>
-  <!-- Joint 5 -->
-  <link name="meca_axis_5_link">
-    <visual>
-      <origin xyz="0 0 0" rpy="0 0 0" />
-      <geometry>
-        <mesh filename="package://mecademic_description/meshes/meca_500_r3_j5.dae" />
-      </geometry>
-    </visual>
-    <collision>
-      <origin xyz="0 0 0" rpy="0 0 0" />
-      <geometry>
-        <mesh filename="package://mecademic_description/meshes/meca_500_r3_j5_collision.stl" />
-      </geometry>
-    </collision>
-  </link>
-  <joint name="meca_axis_5_joint" type="revolute">
-    <origin xyz="0.12 0 0" rpy="0 0 0" />
-    <parent link="meca_axis_4_link" />
-    <child link="meca_axis_5_link" />
-    <axis xyz="0 1 0" />
-    <limit effort="10.0" velocity="5.23599" lower="-2.00713" upper="2.00713" />
-  </joint>
-  <!-- Joint 6 -->
-  <link name="meca_axis_6_link">
-    <visual>
-      <origin xyz="0 0 0" rpy="0 0 0" />
-      <geometry>
-        <mesh filename="package://mecademic_description/meshes/meca_500_r3_j6.dae" />
-      </geometry>
-    </visual>
-    <collision>
-      <origin xyz="0 0 0" rpy="0 0 0" />
-      <geometry>
-        <mesh filename="package://mecademic_description/meshes/meca_500_r3_j6_collision.stl" />
-      </geometry>
-    </collision>
-  </link>
-  <joint name="meca_axis_6_joint" type="revolute">
-    <origin xyz="0.07 0 0" rpy="0 0 0" />
-    <parent link="meca_axis_5_link" />
-    <child link="meca_axis_6_link" />
-    <axis xyz="1 0 0" />
-    <limit effort="10.0" velocity="8.72665" lower="-3.14159" upper="3.14159" />
-  </joint>
-  <!-- FLANGE -->
-  <link name="meca_flange_link" />
-  <joint name="meca_flange_joint" type="fixed">
-    <parent link="meca_axis_6_link" />
-    <child link="meca_flange_link" />
-    <origin xyz="0 0 0" rpy="0 ${pi/2} 0" />
-  </joint>
+<?xml version="1.0"?>
+<robot name="meca_500_r3" xmlns:xacro="http://www.ros.org/wiki/xacro">
+  <!-- Import meca macro -->
+  <xacro:include filename="$(find mecademic_description)/urdf/meca_500_r3.xacro" />
+  <xacro:meca_500_r3
+    prefix=''
+    scale="1.0"
+  />
 </robot>
